Commit message: Align MuJoCo sim with real training environment
Add dual cameras (front + wrist) matching the real SO-ARM101 training
setup, update scene to match training conditions (bowl, single blue
cube, dark mat), and set camera resolution to 640x480.

Camera changes:
- Rename single "camera" to "front", reposition to match real pole
  mount (61cm above table, 28cm behind workspace center)
- Add "wrist" camera on gripper_link pointing along approach direction
- Both cameras publish at 640x480 matching training resolution
- Topics: /front/image_raw, /wrist/image_raw

Scene changes:
- Replace tray with white bowl (cylinder approximation)
- Replace 3 cubes with single blue cube matching training
- Add dark mat on table matching real workspace surface

File: pai_bringup/mjcf/scene.xml.xacro (robot description, xacro)
@@ -39,8 +39,7 @@
     <material name="table_leg" rgba="0.82 0.84 0.86 1" />
     <material name="table_top" rgba="0.18 0.18 0.2 1" reflectance="0.12" />
-    <material name="tray" rgba="0.95 0.95 0.96 1" reflectance="0.2" />
-    <material name="cube_small" rgba="0.9 0.3 0.2 1" />
-    <material name="cube_medium" rgba="0.2 0.7 0.4 1" />
-    <material name="cube_large" rgba="0.2 0.4 0.9 1" />
+    <material name="mat_surface" rgba="0.12 0.12 0.14 1" reflectance="0.05" />
+    <material name="bowl" rgba="0.95 0.95 0.96 1" reflectance="0.2" />
+    <material name="cube_blue" rgba="0.2 0.4 0.9 1" />
   </asset>
   <worldbody>
@@ -54,23 +53,21 @@
       <geom name="leg_br" type="box" pos="0.315 -0.285 -0.1965" size="0.015 0.015 0.1835" material="table_leg" />
     </body>
-    <body name="tray" pos="$(arg tray_x) $(arg tray_y) $(arg tray_z)" euler="$(arg tray_yaw) $(arg tray_pitch) $(arg tray_roll)">
-      <!-- Tray 120x160x20mm: short edge (120mm) along x, long edge (160mm) along y facing arm -->
-      <geom name="tray_floor" type="box" size="0.06 0.08 0.0015" material="tray" friction="0.7 0.1 0.1" />
-      <geom name="tray_wall_f" type="box" pos="0 0.0785 0.0115" size="0.06 0.003 0.01" material="tray" />
-      <geom name="tray_wall_b" type="box" pos="0 -0.0785 0.0115" size="0.06 0.003 0.01" material="tray" />
-      <geom name="tray_wall_l" type="box" pos="-0.0585 0 0.0115" size="0.003 0.08 0.01" material="tray" />
-      <geom name="tray_wall_r" type="box" pos="0.0585 0 0.0115" size="0.003 0.08 0.01" material="tray" />
+    <!-- Dark mat on table (matches real WOWROBOT mat) -->
+    <body name="mat" pos="$(arg tray_x) $(arg tray_y) $(arg tray_z)">
+      <geom name="mat_surface" type="box" size="0.18 0.14 0.001" material="mat_surface" friction="0.7 0.1 0.1" />
     </body>
-    <body name="cube_small" pos="$(arg cube_small_x) $(arg cube_small_y) $(arg cube_small_z)">
-      <freejoint name="cube_small_joint" />
-      <geom name="cube_small_geom" type="box" size="0.0125 0.0125 0.0125" mass="0.02" material="cube_small" friction="0.7 0.1 0.1" />
+    <!-- Bowl: white ceramic, ~12cm diameter, ~6cm tall (matches real setup) -->
+    <body name="bowl" pos="$(arg tray_x) $(arg tray_y) $(arg tray_z)">
+      <!-- Bowl approximated as a cylinder with open top -->
+      <geom name="bowl_base" type="cylinder" size="0.055 0.002" material="bowl" friction="0.7 0.1 0.1" />
+      <geom name="bowl_wall" type="cylinder" size="0.06 0.03" pos="0 0 0.03" material="bowl"
+            friction="0.7 0.1 0.1" contype="1" conaffinity="1" shellinertia="true" />
+      <geom name="bowl_inner" type="cylinder" size="0.052 0.028" pos="0 0 0.032"
+            contype="0" conaffinity="0" group="3" rgba="0 0 0 0" />
     </body>
-    <body name="cube_medium" pos="$(arg cube_medium_x) $(arg cube_medium_y) $(arg cube_medium_z)">
-      <freejoint name="cube_medium_joint" />
-      <geom name="cube_medium_geom" type="box" size="0.0156 0.0156 0.0156" mass="0.04" material="cube_medium" friction="0.7 0.1 0.1" />
-    </body>
-    <body name="cube_large" pos="$(arg cube_large_x) $(arg cube_large_y) $(arg cube_large_z)">
-      <freejoint name="cube_large_joint" />
-      <geom name="cube_large_geom" type="box" size="0.0188 0.0188 0.0188" mass="0.08" material="cube_large" friction="0.7 0.1 0.1" />
+    <!-- Single blue cube (matches real training scene) -->
+    <body name="cube_blue" pos="$(arg cube_large_x) $(arg cube_large_y) $(arg cube_large_z)">
+      <freejoint name="cube_blue_joint" />
+      <geom name="cube_blue_geom" type="box" size="0.0125 0.0125 0.0125" mass="0.02" material="cube_blue" friction="0.7 0.1 0.1" />
     </body>
   </worldbody>

File: pai_bringup/mjcf/so_arm101.xml.xacro (robot description, xacro)
@@ -364,4 +364,7 @@
                   quat="0.707107 -0 0.707107 -2.37788e-17"
                 />
+                <!-- Wrist camera: mounted on gripper, looking forward/down along approach direction -->
+                <site name="wrist_camera_frame" pos="0.0 0.0 -0.05" euler="1.5708 0 0"/>
+                <camera name="wrist" fovy="58" mode="fixed" resolution="640 480" pos="0.0 0.0 -0.05" euler="1.5708 0 0"/>
                 <!-- Link jaw -->
                 <body
@@ -402,7 +405,8 @@
         </body>
       </body>
-      <!-- Camera: elevated above workspace for full scene visibility (table, tray, cubes, gripper) -->
-      <site name="camera_color_mujoco_frame" pos="0.25 0.0 0.55" euler="0 -0.7 0"/>
-      <camera name="camera" fovy="52" mode="fixed" resolution="1280 720" pos="0.25 0.0 0.55" euler="0 -0.7 0"/>
+      <!-- Front camera: matches real setup — on a pole 61cm above table, 28cm behind workspace center.
+           Position is relative to base_link (which has 180° yaw, so local +x = world -x). -->
+      <site name="front_camera_frame" pos="-0.05 0.0 0.6" euler="0 -0.43 0"/>
+      <camera name="front" fovy="58" mode="fixed" resolution="640 480" pos="-0.05 0.0 0.6" euler="0 -0.43 0"/>
     </body>
   </worldbody>

File: pai_bringup/urdf/so_arm101_mujoco.urdf.xacro (robot description, xacro)
@@ -15,10 +15,17 @@
     x="$(arg arm_base_x)" y="$(arg arm_base_y)" z="$(arg arm_base_z)"
     roll="$(arg arm_base_roll)" pitch="$(arg arm_base_pitch)" yaw="$(arg arm_base_yaw)" />
-  <!-- Overhead camera link -->
-  <link name="camera_color_mujoco_frame"/>
-  <joint name="camera_color_mujoco_joint" type="fixed">
+  <!-- Front camera: on a pole behind the workspace, looking steeply down -->
+  <link name="front_camera_frame"/>
+  <joint name="front_camera_joint" type="fixed">
     <parent link="base_link"/>
-    <child link="camera_color_mujoco_frame"/>
-    <origin xyz="0.0 0.0 0.5" rpy="0 2.356 0.0"/>
+    <child link="front_camera_frame"/>
+    <origin xyz="-0.05 0.0 0.6" rpy="0 0 0"/>
+  </joint>
+  <!-- Wrist camera: mounted on gripper, looking forward along approach direction -->
+  <link name="wrist_camera_frame"/>
+  <joint name="wrist_camera_joint" type="fixed">
+    <parent link="gripper_link"/>
+    <child link="wrist_camera_frame"/>
+    <origin xyz="0.0 0.0 -0.05" rpy="0 0 0"/>
   </joint>
   <!-- ros2_control information including camera sensor -->
@@ -84,10 +91,17 @@
       <state_interface name="velocity" />
     </joint>
-    <!-- Camera informatiom -->
-    <sensor name="camera">
-      <param name="frame_name">camera_color_mujoco_frame</param>
-      <param name="info_topic">/camera/info</param>
-      <param name="image_topic">/camera</param>
-      <param name="depth_topic">/camera/depth</param>
+    <!-- Front camera (name must match MJCF <camera name="front">) -->
+    <sensor name="front">
+      <param name="frame_name">front_camera_frame</param>
+      <param name="info_topic">/front/camera_info</param>
+      <param name="image_topic">/front/image_raw</param>
+      <param name="depth_topic">/front/depth</param>
+    </sensor>
+    <!-- Wrist camera (name must match MJCF <camera name="wrist">) -->
+    <sensor name="wrist">
+      <param name="frame_name">wrist_camera_frame</param>
+      <param name="info_topic">/wrist/camera_info</param>
+      <param name="image_topic">/wrist/image_raw</param>
+      <param name="depth_topic">/wrist/depth</param>
     </sensor>
   </ros2_control>
